Commit message: Ajout d'un contact sensor et plugin associé

File: robotino3_description/urdf/robotino_body.xacro (robot description, xacro)
@@ -73,16 +73,16 @@
         </geometry>
       </visual> -->
-<!--       <collision>
+      <collision>
         <origin xyz="0 0 ${BASE_HEIGHT/2+0.02}" rpy="0 0 0" />
         <geometry>
           <cylinder radius="${BASE_RADIUS}" length="${BASE_HEIGHT}"/>
         </geometry>
-      </collision> -->
-      <collision>
+      </collision>
+<!--       <collision>
         <origin xyz="0.01 0 0" rpy="0 0 ${M_PI/2}"/>
         <geometry>
           <mesh filename="package://robotino3_description/meshes/RobotinoBody.dae" scale="${M_SCALE} ${M_SCALE} ${M_SCALE}"/>
         </geometry>
-      </collision>
+      </collision> -->
     </link>
     <wheel name="wheel1" parent="base_link">
@@ -98,5 +98,5 @@
       <axis xyz="1 0 0"/>
     </wheel>
-   <!--  <command_bridge name="command_bridge" parent="base_link">
+    <command_bridge name="command_bridge" parent="base_link">
       <origin xyz="-0.05 0 0.13" rpy="0 0 ${M_PI/2}"/>
     </command_bridge>
@@ -104,13 +104,13 @@
       <origin xyz="0.044 0 0.07" rpy="0 0 ${M_PI/2}"/>
     </camera>
-    <anglebracketusb name="anglebracketusb" parent="base_link">
+<!--     <anglebracketusb name="anglebracketusb" parent="base_link">
       <origin xyz="0.008 0 0.137" rpy="0 0 ${M_PI/2}"/>
     </anglebracketusb> -->
-    <!-- <laser name="laser" parent="base_link">
+<!--     <laser name="laser" parent="base_link">
       <origin xyz="-0.022 0 0.232" rpy="0 0 0"/>
     </laser> -->
-<!--     <laser name="laser" parent="base_link">
+    <laser name="laser" parent="base_link">
       <origin xyz="0.12 0 ${BASE_HEIGHT/2}" rpy="0 0 0"/>
-    </laser> -->
+    </laser>
   </macro>
 </robot>

File: robotino3_description/urdf/robotino_hardware.xacro (robot description, xacro)
@@ -59,10 +59,10 @@
           izz="1.0" />
       </inertial>
-<!--       <collision>
+      <collision>
         <origin xyz="0 0 0" rpy="0 0 0" />
         <geometry>
           <box size="0.25 0.11 0.16"/>
         </geometry>
-      </collision> -->
+      </collision>
     </link>
   </macro>
@@ -82,16 +82,16 @@
           izz="1.0" />
       </inertial>
-<!--       <visual>
+      <visual>
         <origin xyz="0 0 0" rpy="0 0 ${M_PI/2}" />
         <geometry>
           <mesh filename="package://robotino3_description/meshes/RobotinoLaserScanner.dae" scale="${M_SCALE} ${M_SCALE} ${M_SCALE}"/>
         </geometry>
-      </visual> -->
-<!--       <collision>
+      </visual>
+      <collision>
         <origin xyz="0 0 ${HOKUYO_LENGTH/2}" rpy="0 0 0" />
         <geometry>
           <cylinder radius="${HOKUYO_RADIUS}" length="${HOKUYO_LENGTH}" />
         </geometry>
-      </collision> -->
+      </collision>
     </link>
   </macro>
@@ -111,10 +111,10 @@
           izz="1.0" />
       </inertial>
-<!--       <visual>
+      <visual>
         <origin xyz="0 0 0" rpy="0 0 0" />
         <geometry>
           <mesh filename="package://robotino3_description/meshes/RobotinoCamera.dae" scale="${M_SCALE} ${M_SCALE} ${M_SCALE}"/>
         </geometry>
-      </visual> -->
+      </visual>
     </link>
   </macro>
@@ -134,10 +134,10 @@
           izz="1.0" />
       </inertial>
-<!--       <visual>
+      <visual>
         <origin xyz="0 0 0" rpy="0 0 0" />
         <geometry>
           <mesh filename="package://robotino3_description/meshes/AngleBracketUSBHub.dae" scale="${M_SCALE} ${M_SCALE} ${M_SCALE}"/>
         </geometry>
-      </visual> -->
+      </visual>
     </link>
   </macro>
@@ -159,5 +159,5 @@
           izz="1.0" />
       </inertial>
-<!--       <visual>
+      <visual>
         <origin xyz="0 0 0" rpy="0 0 0" />
         <geometry>
@@ -165,5 +165,5 @@
         </geometry>
         <material name="${color}"/>
-      </visual> -->
+      </visual>
       <collision>
         <origin xyz="0 0 0" rpy="0 0 0" />

Commit message: Ajout LaserScan, Camera et Odometry

File: robotino3_description/urdf/robotino_body.xacro (robot description, xacro)
@@ -101,7 +101,7 @@
       <origin xyz="-0.05 0 0.13" rpy="0 0 ${M_PI/2}"/>
     </command_bridge>
-    <camera name="camera" parent="base_link">
-      <origin xyz="0.044 0 0.07" rpy="0 0 ${M_PI/2}"/>
-    </camera>
+    <camera_macro name="camera" parent="base_link">
+      <origin xyz="0.044 0 0.15" rpy="0 0 0"/> <!-- ${M_PI/2} -->
+    </camera_macro>
 <!--     <anglebracketusb name="anglebracketusb" parent="base_link">
       <origin xyz="0.008 0 0.137" rpy="0 0 ${M_PI/2}"/>

File: robotino3_description/urdf/robotino_hardware.xacro (robot description, xacro)
@@ -97,5 +97,5 @@
   </macro>
   <!-- Camera -->
-  <macro name="camera" params="parent name *origin">
+  <macro name="camera_macro" params="parent name *origin">
     <joint name="${name}_joint" type="fixed">
       <insert_block name="origin" />
@@ -140,4 +140,10 @@
         </geometry>
       </visual>
+      <visual>
+        <origin xyz="0 0 0" rpy="0 0 0" />
+        <geometry>
+          <cylinder radius="${HOKUYO_RADIUS}" length="${HOKUYO_LENGTH}" />
+        </geometry>
+      </visual>
     </link>
   </macro>
